Commit message: Created a new urdf for the test_bed

File: description/robot.urdf.xacro (robot description, xacro)
@@ -2,5 +2,5 @@
 <robot xmlns:xacro="http://www.ros.org/wiki/xacro"  name="robot">
     <xacro:include filename="robot_core.xacro"/>
-    <xacro:include filename="depth_camera.xacro"/>
+    <!--<xacro:include filename="depth_camera.xacro"/>-->
     <!--<xacro:include filename="urdf_rover.xacro"/>-->
     <!--<xacro:include filename="ros2_control.xacro"/>-->

File: description/robot_core.xacro (robot description, xacro)
@@ -47,12 +47,75 @@
         </xacro:inertial_box>
     </link>
-    <gazebo reference="chassis">
-        <material>Gazebo/White</material>
-    </gazebo>
     <!-- Front Left Wheel Link -->
+    <joint name="wbl" type="continuous">
+        <parent link="chassis"/>
+        <child link="back_left_wheel"/>
+        <origin xyz="0 ${chassis_y / 2} ${chassis_z / 2}" rpy="-${pi / 2} 0 0"/>
+        <axis xyz="0 0 1"/>
+    </joint>
+    <link name="back_left_wheel">
+        <visual>
+            <geometry>
+                <cylinder radius="${wheel_radius}" length="${wheel_length}"/>
+            </geometry>
+            <material name="blue"/>
+        </visual>
+        <collision>
+            <geometry>
+                <cylinder radius="${wheel_radius}" length="${wheel_length}"/>
+            </geometry>
+        </collision>
+        <xacro:inertial_cylinder mass="0.1" length="${wheel_length}" radius="${wheel_radius}">
+            <origin xyz="0 0 0" rpy="0 0 0"/>
+        </xacro:inertial_cylinder>
+    </link>
+    <joint name="wbr" type="continuous">
+        <parent link="chassis"/>
+        <child link="back_right_wheel"/>
+        <origin xyz="0 -${chassis_y / 2} ${chassis_z / 2}" rpy="-${pi / 2} 0 0"/>
+        <axis xyz="0 0 1"/>
+    </joint>
+    <link name="back_right_wheel">
+        <visual>
+            <geometry>
+                <cylinder radius="${wheel_radius}" length="${wheel_length}"/>
+            </geometry>
+            <material name="blue"/>
+        </visual>
+        <collision>
+            <geometry>
+                <cylinder radius="${wheel_radius}" length="${wheel_length}"/>
+            </geometry>
+        </collision>
+        <xacro:inertial_cylinder mass="0.1" length="${wheel_length}" radius="${wheel_radius}">
+            <origin xyz="0 0 0" rpy="0 0 0"/>
+        </xacro:inertial_cylinder>
+    </link>
+    <joint name="wfr" type="continuous">
+        <parent link="chassis"/>
+        <child link="front_right_wheel"/>
+        <origin xyz="${chassis_x} -${chassis_y / 2} ${chassis_z / 2}" rpy="-${pi / 2} 0 0"/>
+        <axis xyz="0 0 1"/>
+    </joint>
+    <link name="front_right_wheel">
+        <visual>
+            <geometry>
+                <cylinder radius="${wheel_radius}" length="${wheel_length}"/>
+            </geometry>
+            <material name="blue"/>
+        </visual>
+        <collision>
+            <geometry>
+                <cylinder radius="${wheel_radius}" length="${wheel_length}"/>
+            </geometry>
+        </collision>
+        <xacro:inertial_cylinder mass="0.1" length="${wheel_length}" radius="${wheel_radius}">
+            <origin xyz="0 0 0" rpy="0 0 0"/>
+        </xacro:inertial_cylinder>
+    </link>
     <joint name="wfl" type="continuous">
-        <parent link="base_link"/>
+        <parent link="chassis"/>
         <child link="front_left_wheel"/>
-        <origin xyz="${wheel_radius + wheel_separation} ${chassis_y / 2} 0" rpy="-${pi / 2} 0 0"/>
+        <origin xyz="${chassis_x} ${chassis_y / 2} ${chassis_z / 2}" rpy="-${pi / 2} 0 0"/>
         <axis xyz="0 0 1"/>
     </joint>
@@ -73,144 +136,24 @@
         </xacro:inertial_cylinder>
     </link>
-    <gazebo reference="front_left_wheel">
-        <material>Gazebo/Blue</material>
-        <mu1 value="0"/>
-        <mu2 value="0"/>
-    </gazebo>
-    <!-- Middle Left Wheel Link -->
-    <joint name="wml" type="continuous">
-        <parent link="base_link"/>
-        <child link="middle_left_wheel"/>
-        <origin xyz="0 ${chassis_y / 2} 0" rpy="-${pi / 2} 0 0"/>
-        <axis xyz="0 0 1"/>
+    <joint name="depth_camera" type="fixed">
+        <parent link="chassis"/>
+        <child link="camera_link"/>
+        <origin xyz="${chassis_x - (camera_width / 2)} 0 ${chassis_z + (camera_height / 2)}" rpy="0 0 0"/>
     </joint>
-    <link name="middle_left_wheel">
+    <link name="camera_link">
         <visual>
             <geometry>
-                <cylinder radius="${wheel_radius}" length="${wheel_length}"/>
+                <box size="${camera_width} ${camera_length} ${camera_height}"/>
             </geometry>
-            <material name="blue"/>
+            <material name="red"/>
         </visual>
         <collision>
             <geometry>
-                <cylinder radius="${wheel_radius}" length="${wheel_length}"/>
+                <box size="${camera_width} ${camera_length} ${camera_height}"/>
             </geometry>
         </collision>
-        <xacro:inertial_cylinder mass="0.1" length="${wheel_length}" radius="${wheel_radius}">
+        <xacro:inertial_box mass="0.1" x="${camera_width}" y="${camera_length}" z="${camera_height}">
             <origin xyz="0 0 0" rpy="0 0 0"/>
-        </xacro:inertial_cylinder>
+        </xacro:inertial_box>
     </link>
-    <gazebo reference="middle_left_wheel">
-        <material>Gazebo/Blue</material>
-    </gazebo>
-    <!-- Back Left Wheel Link -->
-    <joint name="wbl" type="continuous">
-        <parent link="base_link"/>
-        <child link="back_left_wheel"/>
-        <origin xyz="-${wheel_radius + wheel_separation} ${chassis_y / 2} 0" rpy="-${pi / 2} 0 0"/>
-        <axis xyz="0 0 1"/>
-    </joint>
-    <link name="back_left_wheel">
-        <visual>
-            <geometry>
-                <cylinder radius="${wheel_radius}" length="${wheel_length}"/>
-            </geometry>
-            <material name="blue"/>
-        </visual>
-        <collision>
-            <geometry>
-                <cylinder radius="${wheel_radius}" length="${wheel_length}"/>
-            </geometry>
-        </collision>
-        <xacro:inertial_cylinder mass="0.1" length="${wheel_length}" radius="${wheel_radius}">
-            <origin xyz="0 0 0" rpy="0 0 0"/>
-        </xacro:inertial_cylinder>
-    </link>
-    <gazebo reference="back_left_wheel">
-        <material>Gazebo/Blue</material>
-        <mu1 value="0"/>
-        <mu2 value="0"/>
-    </gazebo>
-    <!-- Front Right Wheel Link -->
-    <joint name="wfr" type="continuous">
-        <parent link="base_link"/>
-        <child link="front_right_wheel"/>
-        <origin xyz="${wheel_radius + wheel_separation} -${chassis_y / 2} 0" rpy="-${pi / 2} 0 ${pi}"/>
-        <axis xyz="0 0 -1"/>
-    </joint>
-    <link name="front_right_wheel">
-        <visual>
-            <geometry>
-                <cylinder radius="${wheel_radius}" length="${wheel_length}"/>
-            </geometry>
-            <material name="blue"/>
-        </visual>
-        <collision>
-            <geometry>
-                <cylinder radius="${wheel_radius}" length="${wheel_length}"/>
-            </geometry>
-        </collision>
-        <xacro:inertial_cylinder mass="0.1" length="${wheel_length}" radius="${wheel_radius}">
-            <origin xyz="0 0 0" rpy="0 0 0"/>
-        </xacro:inertial_cylinder>
-    </link>
-    <gazebo reference="front_right_wheel">
-        <material>Gazebo/Blue</material>
-        <mu1 value="0"/>
-        <mu2 value="0"/>
-    </gazebo>
-    <!-- Middle Right Wheel Link -->
-    <joint name="wmr" type="continuous">
-        <parent link="base_link"/>
-        <child link="middle_right_wheel"/>
-        <origin xyz="0 -${chassis_y / 2} 0" rpy="-${pi / 2} 0 ${pi}"/>
-        <axis xyz="0 0 -1"/>
-    </joint>
-    <link name="middle_right_wheel">
-        <visual>
-            <geometry>
-                <cylinder radius="${wheel_radius}" length="${wheel_length}"/>
-            </geometry>
-            <material name="blue"/>
-        </visual>
-        <collision>
-            <geometry>
-                <cylinder radius="${wheel_radius}" length="${wheel_length}"/>
-            </geometry>
-        </collision>
-        <xacro:inertial_cylinder mass="0.1" length="${wheel_length}" radius="${wheel_radius}">
-            <origin xyz="0 0 0" rpy="0 0 0"/>
-        </xacro:inertial_cylinder>
-    </link>
-    <gazebo reference="middle_right_wheel">
-        <material>Gazebo/Blue</material>
-    </gazebo>
-    <!-- Back right Wheel Link -->
-    <joint name="wbr" type="continuous">
-        <parent link="base_link"/>
-        <child link="back_right_wheel"/>
-        <origin xyz="-${wheel_radius + wheel_separation} -${chassis_y / 2} 0" rpy="-${pi / 2} 0 ${pi}"/>
-        <axis xyz="0 0 -1"/>
-    </joint>
-    <link name="back_right_wheel">
-        <visual>
-            <geometry>
-                <cylinder radius="${wheel_radius}" length="${wheel_length}"/>
-            </geometry>
-            <material name="blue"/>
-        </visual>
-        <collision>
-            <geometry>
-                <cylinder radius="${wheel_radius}" length="${wheel_length}"/>
-            </geometry>
-        </collision>
-        <xacro:inertial_cylinder mass="0.1" length="${wheel_length}" radius="${wheel_radius}">
-            <origin xyz="0 0 0" rpy="0 0 0"/>
-        </xacro:inertial_cylinder>
-    </link>
-    <gazebo reference="back_right_wheel">
-        <material>Gazebo/Blue</material>
-        <mu1 value="0"/>
-        <mu2 value="0"/>
-    </gazebo>
 </robot>

File: description/robot_values.xacro (robot description, xacro)
@@ -2,6 +2,6 @@
 <robot xmlns:xacro="http://www.ros.org/wiki/xacro"  name="robot">
     <xacro:property name="chassis_x" value="0.568"/>
-    <xacro:property name="chassis_y" value="0.4464"/>
-    <xacro:property name="chassis_z" value="0.2632"/>
+    <xacro:property name="chassis_y" value="0.360"/>
+    <xacro:property name="chassis_z" value="0.05"/>
     <xacro:property name="wheel_radius" value="0.1016"/>
     <xacro:property name="wheel_length" value="0.09525"/>
@@ -9,3 +9,6 @@
     <xacro:property name="lidar_radius" value="0.05"/>
     <xacro:property name="lidar_height" value="0.04"/>
+    <xacro:property name="camera_length" value="0.09"/>
+    <xacro:property name="camera_width" value="0.025"/>
+    <xacro:property name="camera_height" value="0.025"/>
 </robot>
