Commit message: changed the urdf

File: description/robot_values.xacro (robot description, xacro)
@@ -1,7 +1,7 @@
 <?xml version="1.0"?>
 <robot xmlns:xacro="http://www.ros.org/wiki/xacro"  name="robot">
-    <xacro:property name="chassis_x" value="0.568"/>
-    <xacro:property name="chassis_y" value="0.360"/>
-    <xacro:property name="chassis_z" value="0.05"/>
+    <xacro:property name="chassis_x" value="0.54"/>
+    <xacro:property name="chassis_y" value="0.4"/>
+    <xacro:property name="chassis_z" value="0.14"/>
     <xacro:property name="wheel_radius" value="0.1016"/>
     <xacro:property name="wheel_length" value="0.09525"/>
@@ -11,4 +11,4 @@
     <xacro:property name="camera_length" value="0.09"/>
     <xacro:property name="camera_width" value="0.025"/>
-    <xacro:property name="camera_height" value="0.025"/>
+    <xacro:property name="camera_height" value="0.055"/>
 </robot>
