Commit message: urdf

File: description/robot_core.xacro (robot description, xacro)
@@ -47,5 +47,5 @@
         </xacro:inertial_box>
     </link>
-    <!-- Front Left Wheel Link -->
+    <!-- Back Left Wheel Link -->
     <joint name="wbl" type="continuous">
         <parent link="chassis"/>
@@ -70,4 +70,5 @@
         </xacro:inertial_cylinder>
     </link>
+    <!-- Back Right Wheel Link -->
     <joint name="wbr" type="continuous">
         <parent link="chassis"/>
@@ -92,4 +93,5 @@
         </xacro:inertial_cylinder>
     </link>
+    <!-- Front Right Wheel Link -->
     <joint name="wfr" type="continuous">
         <parent link="chassis"/>
@@ -114,4 +116,5 @@
         </xacro:inertial_cylinder>
     </link>
+    <!-- Front Left Wheel Link -->
     <joint name="wfl" type="continuous">
         <parent link="chassis"/>
@@ -136,5 +139,6 @@
         </xacro:inertial_cylinder>
     </link>
-    <joint name="depth_camera" type="fixed">
+    <!-- Camera -->
+    <joint name="camera_joint" type="fixed">
         <parent link="chassis"/>
         <child link="camera_link"/>

Commit message: update

File: description/robot_core.xacro (robot description, xacro)
@@ -161,3 +161,24 @@
         </xacro:inertial_box>
     </link>
+    <joint name="imu_joint" type="fixed">
+        <parent link="chassis"/>
+        <child link="imu_link"/>
+        <origin xyz="${camera_width / 2} 0 ${chassis_z + (camera_height / 2)}" rpy="0 0 ${pi}"/>
+    </joint>
+    <link name="imu_link">
+        <visual>
+            <geometry>
+                <box size="${camera_width} ${camera_length} ${camera_height}"/>
+            </geometry>
+            <material name="red"/>
+        </visual>
+        <collision>
+            <geometry>
+                <box size="${camera_width} ${camera_length} ${camera_height}"/>
+            </geometry>
+        </collision>
+        <xacro:inertial_box mass="0.1" x="${camera_width}" y="${camera_length}" z="${camera_height}">
+            <origin xyz="0 0 0" rpy="0 0 0"/>
+        </xacro:inertial_box>
+    </link>
 </robot>

Commit message: update

File: description/robot_core.xacro (robot description, xacro)
@@ -164,5 +164,5 @@
         <parent link="chassis"/>
         <child link="imu_link"/>
-        <origin xyz="${camera_width / 2} 0 ${chassis_z + (camera_height / 2)}" rpy="0 0 ${pi}"/>
+        <origin xyz="${chassis_x - (camera_width / 2) - 6.5} 2.5 ${chassis_z + (camera_height / 2)}" rpy="0 0 ${pi}"/>
     </joint>
     <link name="imu_link">

Commit message: feat: 5/31/2024

File: description/robot_core.xacro (robot description, xacro)
@@ -143,5 +143,5 @@
         <parent link="chassis"/>
         <child link="camera_link"/>
-        <origin xyz="${chassis_x - (camera_width / 2)} 0 ${chassis_z + (camera_height / 2)}" rpy="0 0 0"/>
+        <origin xyz="${chassis_x - (camera_width / 2)} 6.25 ${chassis_z + (camera_height / 2)}" rpy="0 ${16 * pi / 180} 0"/>
     </joint>
     <link name="camera_link">

File: description/robot_values.xacro (robot description, xacro)
@@ -1,14 +1,15 @@
 <?xml version="1.0"?>
 <robot xmlns:xacro="http://www.ros.org/wiki/xacro"  name="robot">
-    <xacro:property name="chassis_x" value="0.54"/>
-    <xacro:property name="chassis_y" value="0.4"/>
-    <xacro:property name="chassis_z" value="0.14"/>
-    <xacro:property name="wheel_radius" value="0.1016"/>
-    <xacro:property name="wheel_length" value="0.09525"/>
-    <xacro:property name="wheel_separation" value="${(chassis_x - (wheel_radius * 2)) / 2}"/>
-    <xacro:property name="lidar_radius" value="0.05"/>
-    <xacro:property name="lidar_height" value="0.04"/>
-    <xacro:property name="camera_length" value="0.09"/>
-    <xacro:property name="camera_width" value="0.025"/>
-    <xacro:property name="camera_height" value="0.055"/>
+    <xacro:property name="offset" value="39.3701"/>
+    <xacro:property name="chassis_x" value="24"/>
+    <xacro:property name="chassis_y" value="18"/>
+    <xacro:property name="chassis_z" value="8"/>
+    <xacro:property name="wheel_radius" value="4"/>
+    <xacro:property name="wheel_length" value="4"/>
+    <xacro:property name="wheel_separation" value="30"/>
+    <xacro:property name="lidar_radius" value="${0.05 * offset}"/>
+    <xacro:property name="lidar_height" value="${0.04 * offset}"/>
+    <xacro:property name="camera_length" value="${0.09 * offset}"/>
+    <xacro:property name="camera_width" value="${0.025 * offset}"/>
+    <xacro:property name="camera_height" value="${0.055 * offset}"/>
 </robot>
